File: IO4-QuadOD.sch (EAGLE design)
At the start: 21 parts, among them CON10 5MM, CON3 5MM, CON9 CONNECTOR-I2CLEFT

Commit message: added values for connectors
Parts:
- CON1: value (none) -> 2.1mm
- MCU: value (none) -> Mini
- X1, X2, X3, X4: value (none) -> 0.156
Changed lines of the file:
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@@
 <setting verticaltext="up"/>
 </settings>
-<grid distance="0.1" unitdist="inch" unit="inch" style="lines" multiple="1" display="no" altdistance="0.01" altunitdist="inch" altunit="inch"/>
+<grid distance="100" unitdist="mil" unit="mil" style="dots" multiple="1" display="yes" altdistance="50" altunitdist="mil" altunit="mil"/>
 <layers>
-<layer number="1" name="Top" color="4" fill="1" visible="yes" active="no"/>
-<layer number="2" name="Route2" color="1" fill="3" visible="yes" active="no"/>
-<layer number="3" name="Route3" color="4" fill="3" visible="yes" active="no"/>
-<layer number="14" name="Route14" color="1" fill="6" visible="yes" active="no"/>
-<layer number="15" name="Route15" color="4" fill="6" visible="yes" active="no"/>
-<layer number="16" name="Bottom" color="1" fill="1" visible="yes" active="no"/>
-<layer number="17" name="Pads" color="2" fill="1" visible="yes" active="no"/>
-<layer number="18" name="Vias" color="2" fill="1" visible="yes" active="no"/>
-<layer number="19" name="Unrouted" color="6" fill="1" visible="yes" active="no"/>
-<layer number="20" name="Dimension" color="15" fill="1" visible="yes" active="no"/>
-<layer number="21" name="tPlace" color="7" fill="1" visible="yes" active="no"/>
-<layer number="22" name="bPlace" color="7" fill="1" visible="yes" active="no"/>
-<layer number="23" name="tOrigins" color="15" fill="1" visible="yes" active="no"/>
-<layer number="24" name="bOrigins" color="15" fill="1" visible="yes" active="no"/>
-<layer number="25" name="tNames" color="7" fill="1" visible="yes" active="no"/>
-<layer number="26" name="bNames" color="7" fill="1" visible="yes" active="no"/>
-<layer number="27" name="tValues" color="7" fill="1" visible="yes" active="no"/>
-<layer number="28" name="bValues" color="7" fill="1" visible="yes" active="no"/>
+<layer number="1" name="Top" color="4" fill="1" visible="no" active="no"/>
+<layer number="2" name="Route2" color="1" fill="3" visible="no" active="no"/>
+<layer number="3" name="Route3" color="4" fill="3" visible="no" active="no"/>
+<layer number="14" name="Route14" color="1" fill="6" visible="no" active="no"/>
+<layer number="15" name="Route15" color="4" fill="6" visible="no" active="no"/>
+<layer number="16" name="Bottom" color="1" fill="1" visible="no" active="no"/>
+<layer number="17" name="Pads" color="2" fill="1" visible="no" active="no"/>
+<layer number="18" name="Vias" color="2" fill="1" visible="no" active="no"/>
+<layer number="19" name="Unrouted" color="6" fill="1" visible="no" active="no"/>
+<layer number="20" name="Dimension" color="15" fill="1" visible="no" active="no"/>
+<layer number="21" name="tPlace" color="7" fill="1" visible="no" active="no"/>
+<layer number="22" name="bPlace" color="7" fill="1" visible="no" active="no"/>
+<layer number="23" name="tOrigins" color="15" fill="1" visible="no" active="no"/>
+<layer number="24" name="bOrigins" color="15" fill="1" visible="no" active="no"/>
+<layer number="25" name="tNames" color="7" fill="1" visible="no" active="no"/>
+<layer number="26" name="bNames" color="7" fill="1" visible="no" active="no"/>
+<layer number="27" name="tValues" color="7" fill="1" visible="no" active="no"/>
+<layer number="28" name="bValues" color="7" fill="1" visible="no" active="no"/>
 <layer number="29" name="tStop" color="7" fill="3" visible="no" active="no"/>
 <layer number="30" name="bStop" color="7" fill="6" visible="no" active="no"/>
@@
 <layer number="35" name="tGlue" color="7" fill="4" visible="no" active="no"/>
 <layer number="36" name="bGlue" color="7" fill="5" visible="no" active="no"/>
-<layer number="37" name="tTest" color="7" fill="1" visible="yes" active="no"/>
-<layer number="38" name="bTest" color="7" fill="1" visible="yes" active="no"/>
+<layer number="37" name="tTest" color="7" fill="1" visible="no" active="no"/>
+<layer number="38" name="bTest" color="7" fill="1" visible="no" active="no"/>
 <layer number="39" name="tKeepout" color="4" fill="11" visible="no" active="no"/>
 <layer number="40" name="bKeepout" color="1" fill="11" visible="no" active="no"/>
@@
 <layer number="44" name="Drills" color="7" fill="1" visible="no" active="no"/>
 <layer number="45" name="Holes" color="7" fill="1" visible="no" active="no"/>
-<layer number="46" name="Milling" color="3" fill="1" visible="yes" active="no"/>
-<layer number="47" name="Measures" color="7" fill="1" visible="yes" active="no"/>
-<layer number="48" name="Document" color="7" fill="1" visible="yes" active="no"/>
-<layer number="49" name="Reference" color="7" fill="1" visible="yes" active="no"/>
-<layer number="50" name="dxf" color="7" fill="1" visible="yes" active="no"/>
-<layer number="51" name="tDocu" color="7" fill="1" visible="yes" active="no"/>
-<layer number="52" name="bDocu" color="7" fill="1" visible="yes" active="no"/>
-<layer number="53" name="tGND_GNDA" color="7" fill="9" visible="yes" active="no"/>
-<layer number="54" name="bGND_GNDA" color="1" fill="9" visible="yes" active="no"/>
-<layer number="56" name="wert" color="7" fill="1" visible="yes" active="no"/>
-<layer number="57" name="tCAD" color="7" fill="1" visible="yes" active="no"/>
-<layer number="59" name="tCarbon" color="7" fill="1" visible="yes" active="no"/>
-<layer number="60" name="bCarbon" color="7" fill="1" visible="yes" active="no"/>
+<layer number="46" name="Milling" color="3" fill="1" visible="no" active="no"/>
+<layer number="47" name="Measures" color="7" fill="1" visible="no" active="no"/>
+<layer number="48" name="Document" color="7" fill="1" visible="no" active="no"/>
+<layer number="49" name="Reference" color="7" fill="1" visible="no" active="no"/>
+<layer number="50" name="dxf" color="7" fill="1" visible="no" active="no"/>
+<layer number="51" name="tDocu" color="7" fill="1" visible="no" active="no"/>
+<layer number="52" name="bDocu" color="7" fill="1" visible="no" active="no"/>
+<layer number="53" name="tGND_GNDA" color="7" fill="9" visible="no" active="no"/>
+<layer number="54" name="bGND_GNDA" color="1" fill="9" visible="no" active="no"/>
+<layer number="56" name="wert" color="7" fill="1" visible="no" active="no"/>
+<layer number="57" name="tCAD" color="7" fill="1" visible="no" active="no"/>
+<layer number="59" name="tCarbon" color="7" fill="1" visible="no" active="no"/>
+<layer number="60" name="bCarbon" color="7" fill="1" visible="no" active="no"/>
 <layer number="90" name="Modules" color="5" fill="1" visible="yes" active="yes"/>
 <layer number="91" name="Nets" color="2" fill="1" visible="yes" active="yes"/>
@@
 <part name="P+2" library="supply1" deviceset="V+" device=""/>
 <part name="GND18" library="supply1" deviceset="GND" device=""/>
-<part name="X1" library="SPCoast" deviceset="KK-156-5" device=""/>
-<part name="X2" library="SPCoast" deviceset="KK-156-5" device=""/>
-<part name="X3" library="SPCoast" deviceset="KK-156-5" device=""/>
-<part name="X4" library="SPCoast" deviceset="KK-156-5" device=""/>
+<part name="X1" library="SPCoast" deviceset="KK-156-5" device="" value="0.156"/>
+<part name="X2" library="SPCoast" deviceset="KK-156-5" device="" value="0.156"/>
+<part name="X3" library="SPCoast" deviceset="KK-156-5" device="" value="0.156"/>
+<part name="X4" library="SPCoast" deviceset="KK-156-5" device="" value="0.156"/>
 <part name="GND2" library="supply1" deviceset="GND" device=""/>
 <part name="P+4" library="supply1" deviceset="V+" device=""/>
@@
 <part name="GND4" library="supply1" deviceset="GND" device=""/>
 <part name="P+5" library="supply1" deviceset="V+" device=""/>
-<part name="MCU" library="SPCoast" deviceset="WEMOS-D1" device="V1"/>
+<part name="MCU" library="SPCoast" deviceset="WEMOS-D1" device="V1" value="Mini"/>
 <part name="P+6" library="supply1" deviceset="V+" device=""/>
 <part name="GND5" library="supply1" deviceset="GND" device=""/>
@@
 <part name="CON10" library="SPCoast" deviceset="CONNECTOR-M03" device="5MM-LOCK" value="5MM"/>
 <part name="P+8" library="supply1" deviceset="V+" device=""/>
-<part name="CON1" library="SPCoast" deviceset="CONNECTOR-DC-POWER" device="-RA"/>
+<part name="CON1" library="SPCoast" deviceset="CONNECTOR-DC-POWER" device="-RA" value="2.1mm"/>
 <part name="MT1" library="SPCoast" deviceset="MOUNTINGHOLE" device=""/>
 <part name="MT2" library="SPCoast" deviceset="MOUNTINGHOLE" device=""/>

Commit message: normalized values
Parts:
- BOARD1: value BOARD100X100-NOHOLES -> BOARD
- CON9: value CONNECTOR-I2CLEFT -> (none)
- DCCIN, TK1, TK2, TK3, TK4: value MSTBA2 -> 0.200
- IO4-MASTER, IO4-SLAVE: value RJ12-INV -> RJ12/6
- MCU: value Mini -> Mini-R2
Changed lines of the file:
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@@
 <parts>
 <part name="FRAME1" library="SPCoast" deviceset="DOC-FRAME-LETTER" device=""/>
-<part name="BOARD1" library="SPCoast" deviceset="BOARD" device="100X100-NOHOLES" value="BOARD100X100-NOHOLES"/>
-<part name="DCCIN" library="SPCoast" deviceset="CONNECTOR-MSTBA2-ORIG" device="" value="MSTBA2"/>
-<part name="TK1" library="SPCoast" deviceset="CONNECTOR-MSTBA2-ORIG" device="" value="MSTBA2"/>
-<part name="TK2" library="SPCoast" deviceset="CONNECTOR-MSTBA2-ORIG" device="" value="MSTBA2"/>
-<part name="TK3" library="SPCoast" deviceset="CONNECTOR-MSTBA2-ORIG" device="" value="MSTBA2"/>
-<part name="TK4" library="SPCoast" deviceset="CONNECTOR-MSTBA2-ORIG" device="" value="MSTBA2"/>
-<part name="IO4-SLAVE" library="SPCoast" deviceset="CONNECTOR-IO4" device="INV" value="RJ12-INV"/>
-<part name="IO4-MASTER" library="SPCoast" deviceset="CONNECTOR-IO4" device="INV" value="RJ12-INV"/>
+<part name="BOARD1" library="SPCoast" deviceset="BOARD" device="100X100-NOHOLES" value="BOARD"/>
+<part name="DCCIN" library="SPCoast" deviceset="CONNECTOR-MSTBA2-ORIG" device="" value="0.200"/>
+<part name="TK1" library="SPCoast" deviceset="CONNECTOR-MSTBA2-ORIG" device="" value="0.200"/>
+<part name="TK2" library="SPCoast" deviceset="CONNECTOR-MSTBA2-ORIG" device="" value="0.200"/>
+<part name="TK3" library="SPCoast" deviceset="CONNECTOR-MSTBA2-ORIG" device="" value="0.200"/>
+<part name="TK4" library="SPCoast" deviceset="CONNECTOR-MSTBA2-ORIG" device="" value="0.200"/>
+<part name="IO4-SLAVE" library="SPCoast" deviceset="CONNECTOR-IO4" device="INV" value="RJ12/6"/>
+<part name="IO4-MASTER" library="SPCoast" deviceset="CONNECTOR-IO4" device="INV" value="RJ12/6"/>
 <part name="GND37" library="supply1" deviceset="GND" device=""/>
 <part name="P+9" library="supply1" deviceset="V+" device=""/>
@@
 <part name="GND4" library="supply1" deviceset="GND" device=""/>
 <part name="P+5" library="supply1" deviceset="V+" device=""/>
-<part name="MCU" library="SPCoast" deviceset="WEMOS-D1" device="V1" value="Mini"/>
+<part name="MCU" library="SPCoast" deviceset="WEMOS-D1" device="V1" value="Mini-R2"/>
 <part name="P+6" library="supply1" deviceset="V+" device=""/>
 <part name="GND5" library="supply1" deviceset="GND" device=""/>
@@
 <instance part="FRAME1" gate="FRAME" x="0" y="0"/>
 <instance part="FRAME1" gate="FRAME_CONTENT" x="147.32" y="0"/>
-<instance part="BOARD1" gate="G$1" x="241.3" y="33.02"/>
+<instance part="BOARD1" gate="B" x="241.3" y="33.02"/>
 <instance part="DCCIN" gate="-1" x="27.94" y="167.64"/>
 <instance part="DCCIN" gate="-2" x="27.94" y="172.72"/>
@@
 <instance part="TK4" gate="-1" x="27.94" y="106.68"/>
 <instance part="TK4" gate="-2" x="27.94" y="111.76"/>
-<instance part="IO4-SLAVE" gate="G$1" x="22.86" y="86.36" rot="MR0"/>
-<instance part="IO4-MASTER" gate="G$1" x="38.1" y="86.36" rot="MR0"/>
+<instance part="IO4-SLAVE" gate="J" x="22.86" y="86.36" rot="MR0"/>
+<instance part="IO4-MASTER" gate="J" x="38.1" y="86.36" rot="MR0"/>
 <instance part="GND37" gate="1" x="40.64" y="76.2" smashed="yes">
 <attribute name="VALUE" x="38.1" y="73.66" size="1.778" layer="96"/>
@@
 <attribute name="VALUE" x="176.53" y="81.28" size="1.778" layer="96" rot="R180"/>
 </instance>
-<instance part="CON1" gate="G$1" x="220.98" y="76.2"/>
+<instance part="CON1" gate="J" x="220.98" y="76.2"/>
 <instance part="MT1" gate="MT1" x="142.24" y="5.08"/>
 <instance part="MT2" gate="MT1" x="142.24" y="12.7"/>
@@
 <net name="OD1" class="0">
 <segment>
-<pinref part="IO4-SLAVE" gate="G$1" pin="2"/>
-<pinref part="IO4-MASTER" gate="G$1" pin="2"/>
+<pinref part="IO4-SLAVE" gate="J" pin="2"/>
+<pinref part="IO4-MASTER" gate="J" pin="2"/>
 <wire x1="40.64" y1="88.9" x2="25.4" y2="88.9" width="0.1524" layer="91"/>
 <label x="165.1" y="88.9" size="1.27" layer="95" xref="yes"/>
@@
 <net name="OD2" class="0">
 <segment>
-<pinref part="IO4-SLAVE" gate="G$1" pin="3"/>
-<pinref part="IO4-MASTER" gate="G$1" pin="3"/>
+<pinref part="IO4-SLAVE" gate="J" pin="3"/>
+<pinref part="IO4-MASTER" gate="J" pin="3"/>
 <wire x1="40.64" y1="86.36" x2="25.4" y2="86.36" width="0.1524" layer="91"/>
 <label x="165.1" y="86.36" size="1.27" layer="95" xref="yes"/>
@@
 <net name="OD3" class="0">
 <segment>
-<pinref part="IO4-SLAVE" gate="G$1" pin="4"/>
-<pinref part="IO4-MASTER" gate="G$1" pin="4"/>
+<pinref part="IO4-SLAVE" gate="J" pin="4"/>
+<pinref part="IO4-MASTER" gate="J" pin="4"/>
 <wire x1="40.64" y1="83.82" x2="25.4" y2="83.82" width="0.1524" layer="91"/>
 <label x="165.1" y="83.82" size="1.27" layer="95" xref="yes"/>
@@
 <net name="OD4" class="0">
 <segment>
-<pinref part="IO4-SLAVE" gate="G$1" pin="5"/>
-<pinref part="IO4-MASTER" gate="G$1" pin="5"/>
+<pinref part="IO4-SLAVE" gate="J" pin="5"/>
+<pinref part="IO4-MASTER" gate="J" pin="5"/>
 <wire x1="40.64" y1="81.28" x2="25.4" y2="81.28" width="0.1524" layer="91"/>
 <label x="165.1" y="78.74" size="1.27" layer="95" xref="yes"/>
@@
 <net name="V+" class="0">
 <segment>
-<pinref part="IO4-MASTER" gate="G$1" pin="1"/>
+<pinref part="IO4-MASTER" gate="J" pin="1"/>
 <wire x1="40.64" y1="91.44" x2="40.64" y2="96.52" width="0.1524" layer="91"/>
 <pinref part="P+9" gate="1" pin="V+"/>
@@
 <wire x1="228.6" y1="78.74" x2="228.6" y2="81.28" width="0.1524" layer="91"/>
 <pinref part="P+2" gate="1" pin="V+"/>
-<pinref part="CON1" gate="G$1" pin="1"/>
+<pinref part="CON1" gate="J" pin="1"/>
 </segment>
 <segment>
@@
 <net name="GND" class="0">
 <segment>
-<pinref part="IO4-SLAVE" gate="G$1" pin="6"/>
-<pinref part="IO4-MASTER" gate="G$1" pin="6"/>
+<pinref part="IO4-SLAVE" gate="J" pin="6"/>
+<pinref part="IO4-MASTER" gate="J" pin="6"/>
 <wire x1="40.64" y1="78.74" x2="25.4" y2="78.74" width="0.1524" layer="91"/>
 <pinref part="GND37" gate="1" pin="GND"/>
@@
 </segment>
 <segment>
-<pinref part="CON1" gate="G$1" pin="3"/>
+<pinref part="CON1" gate="J" pin="3"/>
 <pinref part="GND18" gate="1" pin="GND"/>
-<pinref part="CON1" gate="G$1" pin="2"/>
+<pinref part="CON1" gate="J" pin="2"/>
 <wire x1="228.6" y1="76.2" x2="228.6" y2="73.66" width="0.1524" layer="91"/>
 <junction x="228.6" y="73.66"/>
